File: KiCad/02_power_input.kicad_sch (KiCad schematic)
At the start: 11 parts, among them J202 Barrel_Jack_Switch_Pin3Ring

Commit message: First scheme complete
Parts:
- renumbered C206 to C203, C207 to C204, D204 to D202, J202 to J201
Changed lines of the file:
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@@
 		(dnp no)
 		(fields_autoplaced yes)
-		(property "Reference" "#FLG0203"
+		(property "Reference" "#FLG0202"
 			(at 66.04 43.815 0)
 			(effects
@@
 			(project "solderless_breadboard_psu"
 				(path "/daadd221-9750-45f3-8ee2-46422755319d/658a0cff-7fcc-495d-bed5-c165d7999af0"
-					(reference "#FLG0203")
+					(reference "#FLG0202")
 					(unit 1)
 				)
@@
 		(on_board yes)
 		(dnp no)
-		(property "Reference" "#PWR0216"
+		(property "Reference" "#PWR0208"
 			(at 46.99 81.28 0)
 			(effects
@@
 			(project "solderless_breadboard_psu"
 				(path "/daadd221-9750-45f3-8ee2-46422755319d/658a0cff-7fcc-495d-bed5-c165d7999af0"
-					(reference "#PWR0216")
+					(reference "#PWR0208")
 					(unit 1)
 				)
@@
 		(on_board yes)
 		(dnp no)
-		(property "Reference" "C206"
+		(property "Reference" "C203"
 			(at 63.754 86.868 0)
 			(effects
@@
 			(project "solderless_breadboard_psu"
 				(path "/daadd221-9750-45f3-8ee2-46422755319d/658a0cff-7fcc-495d-bed5-c165d7999af0"
-					(reference "C206")
+					(reference "C203")
 					(unit 1)
 				)
@@
 		(dnp no)
 		(fields_autoplaced yes)
-		(property "Reference" "#PWR0203"
+		(property "Reference" "#PWR0201"
 			(at 48.26 44.45 0)
 			(effects
@@
 			(project "solderless_breadboard_psu"
 				(path "/daadd221-9750-45f3-8ee2-46422755319d/658a0cff-7fcc-495d-bed5-c165d7999af0"
-					(reference "#PWR0203")
+					(reference "#PWR0201")
 					(unit 1)
 				)
@@
 		(dnp no)
 		(fields_autoplaced yes)
-		(property "Reference" "#PWR0210"
+		(property "Reference" "#PWR0206"
 			(at 63.5 64.77 0)
 			(effects
@@
 			(project "solderless_breadboard_psu"
 				(path "/daadd221-9750-45f3-8ee2-46422755319d/658a0cff-7fcc-495d-bed5-c165d7999af0"
-					(reference "#PWR0210")
+					(reference "#PWR0206")
 					(unit 1)
 				)
@@
 		(dnp no)
 		(fields_autoplaced yes)
-		(property "Reference" "#PWR0211"
+		(property "Reference" "#PWR0207"
 			(at 81.28 64.77 0)
 			(effects
@@
 			(project "solderless_breadboard_psu"
 				(path "/daadd221-9750-45f3-8ee2-46422755319d/658a0cff-7fcc-495d-bed5-c165d7999af0"
-					(reference "#PWR0211")
+					(reference "#PWR0207")
 					(unit 1)
 				)
@@
 		(on_board yes)
 		(dnp no)
-		(property "Reference" "J202"
+		(property "Reference" "J201"
 			(at 32.258 39.878 0)
 			(effects
@@
 			(project "solderless_breadboard_psu"
 				(path "/daadd221-9750-45f3-8ee2-46422755319d/658a0cff-7fcc-495d-bed5-c165d7999af0"
-					(reference "J202")
+					(reference "J201")
 					(unit 1)
 				)
@@
 		(dnp no)
 		(fields_autoplaced yes)
-		(property "Reference" "#FLG0202"
+		(property "Reference" "#FLG0201"
 			(at 45.72 43.815 0)
 			(effects
@@
 			(project "solderless_breadboard_psu"
 				(path "/daadd221-9750-45f3-8ee2-46422755319d/658a0cff-7fcc-495d-bed5-c165d7999af0"
-					(reference "#FLG0202")
+					(reference "#FLG0201")
 					(unit 1)
 				)
@@
 		(dnp no)
 		(fields_autoplaced yes)
-		(property "Reference" "#PWR0205"
+		(property "Reference" "#PWR0203"
 			(at 81.28 44.45 0)
 			(effects
@@
 			(project "solderless_breadboard_psu"
 				(path "/daadd221-9750-45f3-8ee2-46422755319d/658a0cff-7fcc-495d-bed5-c165d7999af0"
-					(reference "#PWR0205")
+					(reference "#PWR0203")
 					(unit 1)
 				)
@@
 		(dnp no)
 		(fields_autoplaced yes)
-		(property "Reference" "#FLG0209"
+		(property "Reference" "#FLG0206"
 			(at 83.82 80.645 0)
 			(effects
@@
 			(project "solderless_breadboard_psu"
 				(path "/daadd221-9750-45f3-8ee2-46422755319d/658a0cff-7fcc-495d-bed5-c165d7999af0"
-					(reference "#FLG0209")
+					(reference "#FLG0206")
 					(unit 1)
 				)
@@
 		(dnp no)
 		(fields_autoplaced yes)
-		(property "Reference" "#PWR0204"
+		(property "Reference" "#PWR0202"
 			(at 63.5 44.45 0)
 			(effects
@@
 			(project "solderless_breadboard_psu"
 				(path "/daadd221-9750-45f3-8ee2-46422755319d/658a0cff-7fcc-495d-bed5-c165d7999af0"
-					(reference "#PWR0204")
+					(reference "#PWR0202")
 					(unit 1)
 				)
@@
 		(dnp no)
 		(fields_autoplaced yes)
-		(property "Reference" "#PWR0221"
+		(property "Reference" "#PWR0212"
 			(at 81.28 101.6 0)
 			(effects
@@
 			(project "solderless_breadboard_psu"
 				(path "/daadd221-9750-45f3-8ee2-46422755319d/658a0cff-7fcc-495d-bed5-c165d7999af0"
-					(reference "#PWR0221")
+					(reference "#PWR0212")
 					(unit 1)
 				)
@@
 		(dnp no)
 		(fields_autoplaced yes)
-		(property "Reference" "#FLG0204"
+		(property "Reference" "#FLG0203"
 			(at 83.82 43.815 0)
 			(effects
@@
 			(project "solderless_breadboard_psu"
 				(path "/daadd221-9750-45f3-8ee2-46422755319d/658a0cff-7fcc-495d-bed5-c165d7999af0"
-					(reference "#FLG0204")
+					(reference "#FLG0203")
 					(unit 1)
 				)
@@
 		(on_board yes)
 		(dnp no)
-		(property "Reference" "#PWR0217"
+		(property "Reference" "#PWR0209"
 			(at 63.5 81.28 0)
 			(effects
@@
 			(project "solderless_breadboard_psu"
 				(path "/daadd221-9750-45f3-8ee2-46422755319d/658a0cff-7fcc-495d-bed5-c165d7999af0"
-					(reference "#PWR0217")
+					(reference "#PWR0209")
 					(unit 1)
 				)
@@
 		(dnp no)
 		(fields_autoplaced yes)
-		(property "Reference" "#FLG0208"
+		(property "Reference" "#FLG0205"
 			(at 66.04 80.645 0)
 			(effects
@@
 			(project "solderless_breadboard_psu"
 				(path "/daadd221-9750-45f3-8ee2-46422755319d/658a0cff-7fcc-495d-bed5-c165d7999af0"
-					(reference "#FLG0208")
+					(reference "#FLG0205")
 					(unit 1)
 				)
@@
 		(on_board yes)
 		(dnp no)
-		(property "Reference" "#PWR0218"
+		(property "Reference" "#PWR0210"
 			(at 81.28 81.28 0)
 			(effects
@@
 			(project "solderless_breadboard_psu"
 				(path "/daadd221-9750-45f3-8ee2-46422755319d/658a0cff-7fcc-495d-bed5-c165d7999af0"
-					(reference "#PWR0218")
+					(reference "#PWR0210")
 					(unit 1)
 				)
@@
 		(dnp no)
 		(fields_autoplaced yes)
-		(property "Reference" "#PWR0209"
+		(property "Reference" "#PWR0205"
 			(at 46.99 63.5 0)
 			(effects
@@
 			(project "solderless_breadboard_psu"
 				(path "/daadd221-9750-45f3-8ee2-46422755319d/658a0cff-7fcc-495d-bed5-c165d7999af0"
-					(reference "#PWR0209")
+					(reference "#PWR0205")
 					(unit 1)
 				)
@@
 		(dnp no)
 		(fields_autoplaced yes)
-		(property "Reference" "#FLG0205"
+		(property "Reference" "#FLG0204"
 			(at 110.49 43.815 0)
 			(effects
@@
 			(project "solderless_breadboard_psu"
 				(path "/daadd221-9750-45f3-8ee2-46422755319d/658a0cff-7fcc-495d-bed5-c165d7999af0"
-					(reference "#FLG0205")
+					(reference "#FLG0204")
 					(unit 1)
 				)
@@
 		(dnp no)
 		(fields_autoplaced yes)
-		(property "Reference" "#PWR0220"
+		(property "Reference" "#PWR0211"
 			(at 63.5 101.6 0)
 			(effects
@@
 			(project "solderless_breadboard_psu"
 				(path "/daadd221-9750-45f3-8ee2-46422755319d/658a0cff-7fcc-495d-bed5-c165d7999af0"
-					(reference "#PWR0220")
+					(reference "#PWR0211")
 					(unit 1)
 				)
@@
 		(dnp no)
 		(fields_autoplaced yes)
-		(property "Reference" "#PWR0206"
+		(property "Reference" "#PWR0204"
 			(at 113.03 49.53 0)
 			(effects
@@
 			(project "solderless_breadboard_psu"
 				(path "/daadd221-9750-45f3-8ee2-46422755319d/658a0cff-7fcc-495d-bed5-c165d7999af0"
-					(reference "#PWR0206")
+					(reference "#PWR0204")
 					(unit 1)
 				)
@@
 		(dnp no)
 		(fields_autoplaced yes)
-		(property "Reference" "D204"
+		(property "Reference" "D202"
 			(at 99.3775 76.2 0)
 			(effects
@@
 			(project "solderless_breadboard_psu"
 				(path "/daadd221-9750-45f3-8ee2-46422755319d/658a0cff-7fcc-495d-bed5-c165d7999af0"
-					(reference "D204")
+					(reference "D202")
 					(unit 1)
 				)
@@
 		(on_board yes)
 		(dnp no)
-		(property "Reference" "C207"
+		(property "Reference" "C204"
 			(at 81.534 86.868 0)
 			(effects
@@
 			(project "solderless_breadboard_psu"
 				(path "/daadd221-9750-45f3-8ee2-46422755319d/658a0cff-7fcc-495d-bed5-c165d7999af0"
-					(reference "C207")
-					(unit 1)
-				)
+					(reference "C204")
+					(unit 1)
+				)
