File: KiCad/04_buck_boost.kicad_sch (KiCad schematic)
At the start: 19 parts, among them IC401 TLV62569DBVR, U401 TPS61040DBVR

Commit message: First scheme complete
Parts:
- renumbered C208 to C401, C209 to C402, C210 to C403, C401 to C404, C204 to C405, C402 to C406, D203 to D401, D206 to D402, D207 to D403, L201 to L401, L202 to L402, R204 to R401, R202 to R402, R205 to R403, R203 to R404, R207 to R405, R208 to R406

Commit message: Fill BOM table
Parts:
- C401, C402, C404, C406: footprint Capacitor_SMD:C_0805_2012Metric -> Capacitor_SMD:C_0603_1608Metric; Manufacturer Part Number (none) -> CL10A226MP8NUNE; Manufacturer Product Number CL21A226MQQNNNE -> (none)
- C405: Manufacturer Part Number (none) -> CC0603JRNPO9BN300; Manufacturer Product Number CC0603JRNPO9BN300 -> (none)
- D401: Manufacturer Part Number (none) -> JSMSEMI; Manufacturer Product Number SD0603S040S0R2 -> (none)
- IC401: Manufacturer (none) -> Texas Instruments; Manufacturer Part Number (none) -> TLV62569DBVR; Manufacturer_Name Texas Instruments -> (none); Manufacturer_Part_Number TLV62569DBVR -> (none); Mouser Part Number 595-TLV62569DBVR -> (none); Mouser Price/Stock https://www.mouser.co.uk/ProductDetail/Texas-Instruments/TL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 -> (none)
- L401: Manufacturer Part Number (none) -> FXL0630-100-M; Manufacturer Product Number FXL0630-100-M -> (none)
- L402: Manufacturer Part Number (none) -> FXL0630-150-M; Manufacturer Product Number FXL0630-150-M -> (none)
- R401: Manufacturer Part Number (none) -> 0402WGF1003TCE; Manufacturer Product Number 0402WGF1003TCE -> (none)
- R402: footprint Resistor_SMD:R_0805_2012Metric -> Resistor_SMD:R_0402_1005Metric; Manufacturer Viking Tech -> UNI-ROYAL(Uniroyal Elec); Manufacturer Part Number (none) -> 0402WGF1004TCE; Manufacturer Product Number ARG05FTC1004 -> (none)
- R403: Manufacturer Part Number (none) -> 0402WGF2202TCE; Manufacturer Product Number 0402WGF2202TCE -> (none)
- R404: footprint Resistor_SMD:R_0805_2012Metric -> Resistor_SMD:R_0402_1005Metric; Manufacturer (none) -> UNI-ROYAL(Uniroyal Elec); Manufacturer Part Number (none) -> 0402WGF3303TCE
- U401: Manufacturer (none) -> Texas Instruments; Manufacturer Part Number (none) -> TPS61040DBVR
Changed lines of the file:
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@@
 			)
 		)
-		(property "Footprint" "Capacitor_SMD:C_0805_2012Metric"
+		(property "Footprint" "Capacitor_SMD:C_0603_1608Metric"
 			(at 100.0252 82.55 0)
 			(effects
@@
 			)
 		)
-		(property "Manufacturer Product Number" "CL21A226MQQNNNE"
+		(property "Manufacturer Part Number" "CL10A226MP8NUNE"
 			(at 99.06 78.74 0)
 			(effects
@@
 			)
 		)
-		(property "Footprint" "Capacitor_SMD:C_0805_2012Metric"
+		(property "Footprint" "Capacitor_SMD:C_0603_1608Metric"
 			(at 159.7152 69.85 0)
 			(effects
@@
 			)
 		)
-		(property "Manufacturer Product Number" "CL21A226MQQNNNE"
+		(property "Manufacturer Part Number" "CL10A226MP8NUNE"
 			(at 158.75 66.04 0)
 			(effects
@@
 			)
 		)
-		(property "Manufacturer Product Number" "CC0603JRNPO9BN300 "
+		(property "Manufacturer Part Number" "CC0603JRNPO9BN300"
 			(at 90.17 78.74 0)
 			(effects
@@
 			)
 		)
-		(property "Manufacturer Product Number" "0402WGF1003TCE"
+		(property "Manufacturer Part Number" "0402WGF1003TCE"
 			(at 215.9 66.04 0)
 			(effects
@@
 			)
 		)
-		(property "Footprint" "Capacitor_SMD:C_0805_2012Metric"
+		(property "Footprint" "Capacitor_SMD:C_0603_1608Metric"
 			(at 205.4352 69.85 0)
 			(effects
@@
 			)
 		)
-		(property "Manufacturer Product Number" "CL21A226MQQNNNE"
+		(property "Manufacturer Part Number" "CL10A226MP8NUNE"
 			(at 204.47 66.04 0)
 			(effects
@@
 			)
 		)
-		(property "Footprint" "Capacitor_SMD:C_0805_2012Metric"
+		(property "Footprint" "Capacitor_SMD:C_0603_1608Metric"
 			(at 32.7152 81.28 0)
 			(effects
@@
 			)
 		)
-		(property "Manufacturer Product Number" "CL21A226MQQNNNE"
+		(property "Manufacturer Part Number" "CL10A226MP8NUNE"
 			(at 31.75 77.47 0)
 			(effects
@@
 			)
 		)
+		(property "Manufacturer" "Texas Instruments"
+			(at 41.91 68.58 0)
+			(effects
+				(font
+					(size 1.27 1.27)
+				)
+				(hide yes)
+			)
+		)
+		(property "Manufacturer Part Number" "TPS61040DBVR"
+			(at 41.91 68.58 0)
+			(effects
+				(font
+					(size 1.27 1.27)
+				)
+				(hide yes)
+			)
+		)
 		(pin "5"
 		)
@@
 			)
 		)
-		(property "Manufacturer Product Number" "FXL0630-100-M"
-			(at 46.99 59.69 0)
+		(property "Manufacturer Part Number" "FXL0630-100-M"
+			(at 46.99 59.69 90)
 			(effects
 				(font
@@
 			)
 		)
-		(property "Footprint" "Resistor_SMD:R_0805_2012Metric"
+		(property "Footprint" "Resistor_SMD:R_0402_1005Metric"
 			(at 81.788 77.47 90)
 			(effects
@@
 			)
 		)
-		(property "Manufacturer" "Viking Tech"
+		(property "Manufacturer" "UNI-ROYAL(Uniroyal Elec)"
 			(at 80.01 77.47 0)
 			(effects
@@
 			)
 		)
-		(property "Manufacturer Product Number" "ARG05FTC1004"
+		(property "Manufacturer Part Number" "0402WGF1004TCE"
 			(at 80.01 77.47 0)
 			(effects
@@
 			)
 		)
-		(property "Manufacturer_Name" "Texas Instruments"
-			(at 191.77 552.07 0)
-			(effects
-				(font
-					(size 1.27 1.27)
-				)
-				(justify left top)
-				(hide yes)
-			)
-		)
-		(property "Manufacturer_Part_Number" "TLV62569DBVR"
-			(at 191.77 652.07 0)
-			(effects
-				(font
-					(size 1.27 1.27)
-				)
-				(justify left top)
-				(hide yes)
-			)
-		)
-		(property "Mouser Part Number" "595-TLV62569DBVR"
-			(at 191.77 752.07 0)
-			(effects
-				(font
-					(size 1.27 1.27)
-				)
-				(justify left top)
-				(hide yes)
-			)
-		)
-		(property "Mouser Price/Stock" "https://www.mouser.co.uk/ProductDetail/Texas-Instruments/TLV62569DBVR?qs=0C8XhJW8e4oaylc%252BzBrCmA%3D%3D"
-			(at 191.77 852.07 0)
-			(effects
-				(font
-					(size 1.27 1.27)
-				)
-				(justify left top)
-				(hide yes)
-			)
-		)
 		(property "Arrow Part Number" "TLV62569DBVR"
 			(at 191.77 952.07 0)
@@
 				)
 				(justify left top)
+				(hide yes)
+			)
+		)
+		(property "Manufacturer" "Texas Instruments"
+			(at 170.18 57.15 0)
+			(effects
+				(font
+					(size 1.27 1.27)
+				)
+				(hide yes)
+			)
+		)
+		(property "Manufacturer Part Number" "TLV62569DBVR"
+			(at 170.18 57.15 0)
+			(effects
+				(font
+					(size 1.27 1.27)
+				)
 				(hide yes)
 			)
@@
 			)
 		)
-		(property "Footprint" "Resistor_SMD:R_0805_2012Metric"
+		(property "Footprint" "Resistor_SMD:R_0402_1005Metric"
 			(at 81.788 90.17 90)
 			(effects
@@
 			)
 		)
-		(property "Manufacturer" ""
+		(property "Manufacturer" "UNI-ROYAL(Uniroyal Elec)"
 			(at 80.01 90.17 0)
 			(effects
@@
 			)
 		)
-		(property "Manufacturer Product Number" ""
+		(property "Manufacturer Part Number" "0402WGF3303TCE"
 			(at 80.01 90.17 0)
 			(effects
@@
 			)
 		)
-		(property "Manufacturer Product Number" "0402WGF2202TCE"
+		(property "Manufacturer Part Number" "0402WGF2202TCE"
 			(at 215.9 80.01 0)
 			(effects
@@
 			)
 		)
-		(property "Manufacturer Product Number" "SD0603S040S0R2"
+		(property "Manufacturer Part Number" "JSMSEMI"
 			(at 68.58 71.12 0)
 			(effects
@@
 			)
 		)
-		(property "Manufacturer Product Number" "FXL0630-150-M"
-			(at 199.39 59.69 0)
-			(effects
-				(font
+		(property "Manufacturer Part Number" "FXL0630-150-M"
+			(at 199.39 59.69 90)
+			(effects
+				(font

Commit message: Production files
Parts:
- D401: footprint Diode_SMD:D_0603_1608Metric -> Diode_SMD:D_SMA; Manufacturer Schottky Diode -> BORN; Manufacturer Part Number JSMSEMI -> SS14
Changed lines of the file:
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@@
 			)
 		)
-		(property "Footprint" "Diode_SMD:D_0603_1608Metric"
+		(property "Footprint" "Diode_SMD:D_SMA"
 			(at 68.58 66.675 0)
 			(effects
@@
 			)
 		)
-		(property "Datasheet" "https://www.vishay.com/docs/88746/ss12.pdf"
+		(property "Datasheet" "https://www.lcsc.com/datasheet/C266551.pdf"
 			(at 68.58 71.12 0)
 			(effects
@@
 			)
 		)
-		(property "Description" "40V 1A Schottky Diode, SMA"
+		(property "Description" "Diode 40V 1A Surface Mount SMA(DO-214AC)"
 			(at 68.58 71.12 0)
 			(effects
@@
 			)
 		)
-		(property "Manufacturer" "Schottky Diode"
+		(property "Manufacturer" "BORN"
 			(at 68.58 71.12 0)
 			(effects
@@
 			)
 		)
-		(property "Manufacturer Part Number" "JSMSEMI"
+		(property "Manufacturer Part Number" "SS14"
 			(at 68.58 71.12 0)
 			(effects

Commit message: battery connector update
Parts:
- D401: footprint Diode_SMD:D_SMA -> Diode_SMD:D_0603_1608Metric; Manufacturer BORN -> Schottky Diode; Manufacturer Part Number SS14 -> SD0603S040S0R2
Changed lines of the file:
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@@
 			)
 		)
-		(property "Footprint" "Diode_SMD:D_SMA"
+		(property "Footprint" "Diode_SMD:D_0603_1608Metric"
 			(at 68.58 66.675 0)
 			(effects
@@
 			)
 		)
-		(property "Datasheet" "https://www.lcsc.com/datasheet/C266551.pdf"
+		(property "Datasheet" "https://www.vishay.com/docs/88746/ss12.pdf"
 			(at 68.58 71.12 0)
 			(effects
@@
 			)
 		)
-		(property "Description" "Diode 40V 1A Surface Mount SMA(DO-214AC)"
+		(property "Description" "40V 1A Schottky Diode, SMA"
 			(at 68.58 71.12 0)
 			(effects
@@
 			)
 		)
-		(property "Manufacturer" "BORN"
+		(property "Manufacturer" "Schottky Diode"
 			(at 68.58 71.12 0)
 			(effects
@@
 			)
 		)
-		(property "Manufacturer Part Number" "SS14"
+		(property "Manufacturer Part Number" "SD0603S040S0R2"
 			(at 68.58 71.12 0)
 			(effects

Commit message: BOM updates
Parts:
- D401: Manufacturer Schottky Diode -> Kyocera AVX
- L401, L402: Manufacturer cjiang (Changjiang Microelectronics Tech) -> cjiang
- R401, R403, R405, R406: Manufacturer UNI-ROYAL(Uniroyal Elec) -> UNI-ROYAL
- R402: value 1MR -> 910kR; Manufacturer UNI-ROYAL(Uniroyal Elec) -> UNI-ROYAL; Manufacturer Part Number 0402WGF1004TCE -> 0402WGJ0914TCE
- R404: value 330kR -> 300kR; Manufacturer UNI-ROYAL(Uniroyal Elec) -> UNI-ROYAL; Manufacturer Part Number 0402WGF3303TCE -> 0402WGF3003TCE
Other:
- note added: "Vout = 1.233V * (1+R1/R2) Vout = 1.233V * (1+910/300) Vout = 4.97V"
- note removed: "Vout = 1.233V * (1+R1/R2) Vout = 1.233V * (1+1000/330) Vout = 4.95V"
Changed lines of the file:
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@@
 		)
 	)
-	(text "Vout = 1.233V * (1+R1/R2)\nVout = 1.233V * (1+1000/330)\nVout = 4.95V"
+	(text "Vout = 1.233V * (1+R1/R2)\nVout = 1.233V * (1+910/300)\nVout = 4.97V"
 		(exclude_from_sim no)
 		(at 64.008 56.388 0)
@@
 			)
 		)
-		(property "Manufacturer" "UNI-ROYAL(Uniroyal Elec)"
+		(property "Manufacturer" "UNI-ROYAL"
 			(at 215.9 66.04 0)
 			(effects
@@
 			)
 		)
-		(property "Manufacturer" "cjiang (Changjiang Microelectronics Tech)"
+		(property "Manufacturer" "cjiang"
 			(at 46.99 59.69 0)
 			(effects
@@
 			)
 		)
-		(property "Manufacturer" "UNI-ROYAL(Uniroyal Elec)"
+		(property "Manufacturer" "UNI-ROYAL"
 			(at 20.32 172.72 0)
 			(effects
@@
 			)
 		)
-		(property "Value" "1MR"
-			(at 86.36 78.994 0)
+		(property "Value" "910kR"
+			(at 87.63 78.232 0)
 			(effects
 				(font
@@
 			)
 		)
-		(property "Manufacturer" "UNI-ROYAL(Uniroyal Elec)"
+		(property "Manufacturer" "UNI-ROYAL"
 			(at 80.01 77.47 0)
 			(effects
@@
 			)
 		)
-		(property "Manufacturer Part Number" "0402WGF1004TCE"
+		(property "Manufacturer Part Number" "0402WGJ0914TCE"
 			(at 80.01 77.47 0)
 			(effects
@@
 			)
 		)
-		(property "Manufacturer" "UNI-ROYAL(Uniroyal Elec)"
+		(property "Manufacturer" "UNI-ROYAL"
 			(at 31.75 172.72 0)
 			(effects
@@
 			)
 		)
-		(property "Value" "330kR"
+		(property "Value" "300kR"
 			(at 88.138 90.17 0)
 			(effects
@@
 			)
 		)
-		(property "Manufacturer" "UNI-ROYAL(Uniroyal Elec)"
+		(property "Manufacturer" "UNI-ROYAL"
 			(at 80.01 90.17 0)
 			(effects
@@
 			)
 		)
-		(property "Manufacturer Part Number" "0402WGF3303TCE"
+		(property "Manufacturer Part Number" "0402WGF3003TCE"
 			(at 80.01 90.17 0)
 			(effects
@@
 			)
 		)
-		(property "Manufacturer" "UNI-ROYAL(Uniroyal Elec)"
+		(property "Manufacturer" "UNI-ROYAL"
 			(at 215.9 80.01 0)
 			(effects
@@
 			)
 		)
-		(property "Manufacturer" "Schottky Diode"
+		(property "Manufacturer" "Kyocera AVX"
 			(at 68.58 71.12 0)
 			(effects
@@
 			)
 		)
-		(property "Manufacturer" "cjiang (Changjiang Microelectronics Tech)"
+		(property "Manufacturer" "cjiang"
 			(at 199.39 59.69 0)
 			(effects
