File: KiCad/v2/03_usb2uart.kicad_sch (KiCad schematic)
At the start: 35 parts, among them IC301 CP2102N-A02-GQFN24R, J301 Conn_01x09_Pin, J302 Conn_01x09_Pin, J303 Conn_01x06_Pin, J304 USB_C_Receptacle_USB2.0_16P, J305 Conn_01x03_Pin, U301 USBLC6-2SC6

Commit message: BOM updates
Parts:
- C301, C303, C304, C307, C310, C311: LCSC Part Number C1591 -> C126532; Manufacturer Samsung Electro-Mechanics -> muRata; Manufacturer Part Number CL10B104KB8NNNC -> GCM155R71H102KA37D
- C302, C305, C306: LCSC Part Number C1779 -> C1705; Manufacturer Part Number CL21A475KAQNNNE -> CL10A475KP8NNNC
- C312: LCSC Part Number (none) -> C86295
- D301, D302, D303: LCSC Part Number (none) -> C965799
- D304: LCSC Part Number (none) -> C82544
- IC301: LCSC Part Number (none) -> C969151; Manufacturer (none) -> SILICON LABS; Manufacturer Part Number (none) -> CP2102N-A02-GQFN24R
- R301: LCSC Part Number (none) -> C844504; Manufacturer (none) -> VISHAY; Manufacturer Part Number (none) -> CRCW040222K1FKED
- R302: LCSC Part Number (none) -> C853963; Manufacturer (none) -> YAGEO; Manufacturer Part Number (none) -> RT0402DRE0747K5L
- R303, R306, R307, R308: LCSC Part Number (none) -> C106235; Manufacturer (none) -> YAGEO; Manufacturer Part Number (none) -> RC0402FR-071KL
- R304, R305: LCSC Part Number C122968 -> C852856; Manufacturer Part Number RT0805BRD075K1L -> RT0402BRD075K1L
- R309: LCSC Part Number (none) -> C2765610; Manufacturer (none) -> UNI-ROYAL; Manufacturer Part Number (none) -> CQ02WGF1002TCE
- R310: LCSC Part Number C218408 -> C1883577; Manufacturer Viking Tech -> YAGEO; Manufacturer Part Number ARG05FTC1004 -> RE0402BRE071ML
- SW301: LCSC Part Number (none) -> C29781314; Manufacturer (none) -> SM Switch; Manufacturer Part Number (none) -> SMG-01-H080A1
