File: KiCad/v2/03_usb2uart.kicad_sch (KiCad schematic)
At the start: 35 parts, among them IC301 CP2102N-A02-GQFN24R, J301 Conn_01x09_Pin, J302 Conn_01x09_Pin, J303 Conn_01x06_Pin, J304 USB_C_Receptacle_USB2.0_16P, J305 Conn_01x03_Pin, U301 USBLC6-2SC6

Commit message: preproduction
Parts:
- C301, C303, C304, C307, C310, C311: LCSC Part Number C126532 -> C85858; Manufacturer Part Number GCM155R71H102KA37D -> GCM155R71H104KE02D
- C313: LCSC Part Number C277510 -> C100040; Manufacturer Part Number CC0603KRX7RYBB102 -> CC0603KRX7R9BB102
Changed lines of the file:
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@@
 			)
 		)
-		(property "Manufacturer Part Number" "GCM155R71H102KA37D"
+		(property "Manufacturer Part Number" "GCM155R71H104KE02D"
 			(at 153.67 66.04 90)
 			(effects
@@
 			)
 		)
-		(property "LCSC Part Number" "C126532"
+		(property "LCSC Part Number" "C85858"
 			(at 153.67 66.04 90)
 			(effects
@@
 			)
 		)
-		(property "Manufacturer Part Number" "GCM155R71H102KA37D"
+		(property "Manufacturer Part Number" "GCM155R71H104KE02D"
 			(at 175.26 39.37 90)
 			(effects
@@
 			)
 		)
-		(property "LCSC Part Number" "C126532"
+		(property "LCSC Part Number" "C85858"
 			(at 175.26 39.37 90)
 			(effects
@@
 			)
 		)
-		(property "Manufacturer Part Number" "GCM155R71H102KA37D"
+		(property "Manufacturer Part Number" "GCM155R71H104KE02D"
 			(at 99.06 86.36 90)
 			(effects
@@
 			)
 		)
-		(property "LCSC Part Number" "C126532"
+		(property "LCSC Part Number" "C85858"
 			(at 99.06 86.36 90)
 			(effects
@@
 			)
 		)
-		(property "Manufacturer Part Number" "CC0603KRX7RYBB102"
+		(property "Manufacturer Part Number" "CC0603KRX7R9BB102"
 			(at 33.02 184.15 90)
 			(effects
@@
 			)
 		)
-		(property "LCSC Part Number" "C277510"
+		(property "LCSC Part Number" "C100040"
 			(at 33.02 184.15 90)
 			(effects
@@
 			)
 		)
-		(property "Manufacturer Part Number" "GCM155R71H102KA37D"
+		(property "Manufacturer Part Number" "GCM155R71H104KE02D"
 			(at 116.84 177.8 90)
 			(effects
@@
 			)
 		)
-		(property "LCSC Part Number" "C126532"
+		(property "LCSC Part Number" "C85858"
 			(at 116.84 177.8 90)
 			(effects
@@
 			)
 		)
-		(property "Manufacturer Part Number" "GCM155R71H102KA37D"
+		(property "Manufacturer Part Number" "GCM155R71H104KE02D"
 			(at 158.75 44.45 90)
 			(effects
@@
 			)
 		)
-		(property "LCSC Part Number" "C126532"
+		(property "LCSC Part Number" "C85858"
 			(at 158.75 44.45 90)
 			(effects
@@
 			)
 		)
-		(property "Manufacturer Part Number" "GCM155R71H102KA37D"
+		(property "Manufacturer Part Number" "GCM155R71H104KE02D"
 			(at 175.26 64.77 90)
 			(effects
@@
 			)
 		)
-		(property "LCSC Part Number" "C126532"
+		(property "LCSC Part Number" "C85858"
 			(at 175.26 64.77 90)
 			(effects

Commit message: Production files
Parts:
- R309: LCSC Part Number C2765610 -> C60490; Manufacturer UNI-ROYAL -> YAGEO; Manufacturer Part Number CQ02WGF1002TCE -> RC0402FR-0710KL
Changed lines of the file:
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@@
 			)
 		)
-		(property "Manufacturer" "UNI-ROYAL"
+		(property "Manufacturer" "YAGEO"
 			(at 130.81 162.56 0)
 			(effects
@@
 			)
 		)
-		(property "Manufacturer Part Number" "CQ02WGF1002TCE"
+		(property "Manufacturer Part Number" "RC0402FR-0710KL"
 			(at 130.81 162.56 0)
 			(effects
@@
 			)
 		)
-		(property "LCSC Part Number" "C2765610"
+		(property "LCSC Part Number" "C60490"
 			(at 130.81 162.56 0)
 			(effects
