File: KiCad/v2/02_power.kicad_sch (KiCad schematic)
At the start: 45 parts, among them IC201 TPS63000DRCR, IC202 TPS63000DRCR, J201 Conn_01x02_Pin, J202 Conn_01x03_Pin, J203 Conn_02x03_Odd_Even, J204 Conn_01x03_Pin, J205 Conn_02x03_Odd_Even

Commit message: BOM updates
Parts:
- C201, C202, C208, C209: LCSC Part Number (none) -> C23630
- C203, C205, C206, C210, C212, C213: LCSC Part Number (none) -> C91606; Manufacturer (none) -> muRata; Manufacturer Part Number (none) -> GRM188R61E106MA73D
- C204: LCSC Part Number (none) -> C113797
- C207, C214: LCSC Part Number C1591 -> C126532; Manufacturer Samsung Electro-Mechanics -> muRata; Manufacturer Part Number CL10B104KB8NNNC -> GCM155R71H102KA37D
- C211: Manufacturer YAGEO -> (none); Manufacturer Part Number CC0603JRNPO9BN300 -> (none)
- C215, C216: LCSC Part Number (none) -> C86295
- D201, D203, D205, D206: LCSC Part Number (none) -> C82544
- D202, D204: LCSC Part Number (none) -> C965799
- F201, F202: LCSC Part Number (none) -> C883112
- FB201, FB202, FB203, FB204: LCSC Part Number (none) -> C14709
- IC201, IC202: LCSC Part Number (none) -> C116655; Manufacturer (none) -> TI; Manufacturer Part Number (none) -> TPS63002DRCR
- L201, L202: LCSC Part Number (none) -> C167218; Manufacturer (none) -> cjiang; Manufacturer Part Number (none) -> FXL0630-2R2-M
- R201, R205: LCSC Part Number (none) -> C106235; Manufacturer (none) -> YAGEO; Manufacturer Part Number (none) -> RC0402FR-071KL
- R202, R206: LCSC Part Number (none) -> C705627; Manufacturer (none) -> YAGEO; Manufacturer Part Number (none) -> RT0402BRD07100RL
- R203: value 900kR -> 910kR; LCSC Part Number (none) -> C2909391; Manufacturer (none) -> FOJAN; Manufacturer Part Number (none) -> FRC0402F9103TS
- R204, R208: LCSC Part Number (none) -> C852472; Manufacturer (none) -> YAGEO; Manufacturer Part Number (none) -> RT0402BRD07100KL
- R207: LCSC Part Number (none) -> C132339; Manufacturer (none) -> UNI-ROYAL; Manufacturer Part Number (none) -> 0402WGF5603TCE

Commit message: preproduction
Parts:
- C204: LCSC Part Number C113797 -> C519102; Manufacturer Part Number CC0603JRNPO9BN300 -> CC0603BRNPO9BN2R4
- C207, C214: LCSC Part Number C126532 -> C85858; Manufacturer Part Number GCM155R71H102KA37D -> GCM155R71H104KE02D
Changed lines of the file:
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@@
 			)
 		)
-		(property "Manufacturer Part Number" "GCM155R71H102KA37D"
+		(property "Manufacturer Part Number" "GCM155R71H104KE02D"
 			(at 163.83 67.31 90)
 			(effects
@@
 			)
 		)
-		(property "LCSC Part Number" "C126532"
+		(property "LCSC Part Number" "C85858"
 			(at 163.83 67.31 90)
 			(effects
@@
 			)
 		)
-		(property "Manufacturer Part Number" "GCM155R71H102KA37D"
+		(property "Manufacturer Part Number" "GCM155R71H104KE02D"
 			(at 163.83 130.81 90)
 			(effects
@@
 			)
 		)
-		(property "LCSC Part Number" "C126532"
+		(property "LCSC Part Number" "C85858"
 			(at 163.83 130.81 90)
 			(effects
@@
 			)
 		)
-		(property "Manufacturer Part Number" "CC0603JRNPO9BN300"
+		(property "Manufacturer Part Number" "CC0603BRNPO9BN2R4"
 			(at 223.52 57.15 0)
 			(effects
@@
 			)
 		)
-		(property "LCSC Part Number" "C113797"
+		(property "LCSC Part Number" "C519102"
 			(at 223.52 57.15 0)
 			(effects
