File: KiCad/v2/solderless_breadboard_psu.kicad_pcb (KiCad board)
At the start: 4 copper layers, 53 x 51 mm, 78 parts, among them IC201 TPS63000DRCR, IC202 TPS63000DRCR, IC301 CP2102N-A02-GQFN24R, J201 Conn_01x02_Pin, J202 Conn_01x03_Pin, J203 Conn_02x03_Odd_Even, J204 Conn_01x03_Pin, J205 Conn_02x03_Odd_Even, J301 Conn_01x09_Pin, J302 Conn_01x09_Pin, J303 Conn_01x06_Pin, J304 USB_C_Receptacle_USB2.0_16P, J305 Conn_01x03_Pin, U301 USBLC6-2SC6

Commit message: BOM updates
Parts:
- R203: value 900kR -> 910kR
- moved R205 0.25 mm to (74.5, 78.5)

Commit message: preproduction
Changed lines of the file:
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@@
 	)
 	(segment
-		(start 72.25 56.75)
-		(end 72.975 56.75)
-		(width 0.7)
-		(layer "F.Cu")
-		(net 2)
-	)
-	(segment
 		(start 78.5 63.4625)
 		(end 79.7125 63.4625)
@@
 	)
 	(segment
+		(start 72.975 56.025)
+		(end 72.975 56.75)
+		(width 0.7)
+		(layer "F.Cu")
+		(net 2)
+	)
+	(segment
 		(start 67.5 87.775)
 		(end 67.5 89)
@@
 	)
 	(segment
+		(start 73.2 55.8)
+		(end 72.975 56.025)
+		(width 0.7)
+		(layer "F.Cu")
+		(net 2)
+	)
+	(segment
 		(start 84.525 97.275)
 		(end 84.525 98)
@@
 	)
 	(via
-		(at 78.5 79.75)
+		(at 78.6 79.75)
 		(size 0.7)
 		(drill 0.3)
@@
 	)
 	(via
-		(at 72.25 56.75)
+		(at 73.2 55.8)
 		(size 0.7)
 		(drill 0.3)
@@
 	)
 	(via
-		(at 80.25 79.75)
+		(at 80.4 79.75)
 		(size 0.7)
 		(drill 0.3)
@@
 	)
 	(segment
-		(start 83.125 73.25)
-		(end 83.75 73.25)
+		(start 77.25 75)
+		(end 77.75 75.5)
 		(width 0.3)
 		(layer "F.Cu")
@@
 	)
 	(segment
-		(start 77.25 75)
-		(end 77.75 75.5)
+		(start 79.5 78.225)
+		(end 80.25 77.475)
 		(width 0.3)
 		(layer "F.Cu")
@@
 	)
 	(segment
-		(start 79.5 78.225)
-		(end 80.25 77.475)
+		(start 82.5 72.625)
+		(end 82.635 72.76)
+		(width 0.3)
+		(layer "F.Cu")
+		(net 15)
+	)
+	(segment
+		(start 82.635 72.76)
+		(end 83.75 72.76)
 		(width 0.3)
 		(layer "F.Cu")
@@
 	)
 	(segment
-		(start 82.5 72.625)
-		(end 83.125 73.25)
+		(start 79.77 75.52)
+		(end 79.5 75.52)
 		(width 0.3)
 		(layer "F.Cu")
@@
 	)
 	(segment
-		(start 79.77 75.52)
-		(end 79.5 75.52)
+		(start 82.5 72.25)
+		(end 82.5 72.625)
 		(width 0.3)
 		(layer "F.Cu")
@@
 	)
 	(segment
-		(start 82.5 72.25)
-		(end 82.5 72.625)
-		(width 0.3)
-		(layer "F.Cu")
-		(net 15)
-	)
-	(segment
 		(start 82.75 66.5)
 		(end 82.5 66.25)
@@
 	)
 	(segment
-		(start 74.1 93.255)
-		(end 74.1 90.7875)
+		(start 78.9 88.35)
+		(end 78.9 90.7)
 		(width 0.7)
 		(layer "F.Cu")
@@
 	)
 	(segment
-		(start 78.9 88.35)
+		(start 78.9 90.7)
 		(end 78.9 93.255)
-		(width 0.7)
+		(width 0.5)
+		(layer "F.Cu")
+		(net 30)
+	)
+	(segment
+		(start 74.1 93.255)
+		(end 74.1 90.7875)
+		(width 0.5)
 		(layer "F.Cu")
 		(net 30)
@@
 	)
 	(segment
+		(start 79.25 88)
+		(end 78.9 88.35)
+		(width 0.7)
+		(layer "F.Cu")
+		(net 30)
+	)
+	(segment
 		(start 74.1 90.7875)
 		(end 72.28125 88.96875)
@@
 		(width 0.7)
 		(layer "F.Cu")
-		(net 30)
-	)
-	(segment
-		(start 79.25 88)
-		(end 78.9 88.35)
-		(width 0.7)
-		(layer "F.Cu")
